File: Micro-Mouse Power Subsystem.kicad_sch (KiCad schematic)
At the start: 81 parts, among them J1 Pin Header, J2 TYPE-C-31-M-12, J3 Conn_01x02, Q1 2N7002, Q2 AO3401A, Q3 AO3400A, Q4 AO3400A, Q5 AO3401A, SW1 SW_SPDT, U1 TP4056-42-ESOP8, U2 brushed DC motors, U3 auxiliary motors, U4 HUSB237-AA001-DN06R, U5 TPS61088RHLR, U6 INA219AIDCNR, U7 XL1509-3.3, U8 XL1509-5.0

Commit message: Added footprints and adjusted labelling
Parts:
- C10, C_{1}1, C_{BOOT}1, C_{BYPASS}1, C_{BY}1, C_{COMP}1, C_{IN_5}1, C_{SS}1: footprint (none) -> Capacitor_SMD:C_0805_2012Metric
- C_{CHARGE_IN}1, C_{CHARGE_OUT}1, C_{IN_3.3}3, C_{OUT}4, C_{OUT}5, C_{OUT}6: footprint (none) -> Capacitor_SMD:C_0603_1608Metric
- C_{IN_3.3}1, C_{IN_3.3}2, C_{IN}3, C_{OUT_3.3}1, C_{OUT_3.3}2, C_{OUT_3.3}3, C_{OUT}3: footprint (none) -> Capacitor_SMD:C_1206_3216Metric
- C_{IN}1, C_{IN}2, C_{OUT}1, C_{OUT}2: footprint (none) -> Capacitor_SMD:C_1210_3225Metric
- L1: footprint (none) -> Inductor_SMD:L_0805_2012Metric
- R_{COMP}1, R_{FB}1, R_{FB}2, R_{FSW}1, R_{FSW}2, R_{ILIM}1, R_{SCL}1, R_{SDA}1: footprint (none) -> Resistor_SMD:R_0805_2012Metric
- R_{LIMIT}1, R_{PROG}1, R_{PROG}2, R_{PULL_DOWN}1: footprint (none) -> Resistor_SMD:R_0603_1608Metric
- R_{SHUNT}1: value 0.05 -> 0.075; footprint (none) -> Resistor_SMD:R_0805_2012Metric
Connections:
- net 3V3_OUT is gone; now on net 3.3V_OUT: C_{BYPASS}1.2, U6.8 (A1)
- net Switch_out is gone; now on net SWITCH_OUT: SW1.3 (C)
- net Battery : no longer SW1.2 (B)
- net GND: now also C10.2, C_{1}1.2, C_{IN_3.3}1.2, C_{IN_3.3}2.2, C_{IN_3.3}3.2, C_{IN}1.2, C_{IN}2.2, C_{IN}3.2, C_{OUT_3.3}1.2, C_{OUT_3.3}2.2, C_{OUT_3.3}3.2, C_{OUT}1.2, C_{OUT}2.2, C_{OUT}3.2, D3.2 (A), D4.2 (A), J3.1 (Pin_1), U7.4 (~{EN}), U7.5 (GND), U7.6 (GND), U7.7 (GND), U7.8 (GND), U8.4 (~{EN}), U8.5 (GND), U8.6 (GND), U8.7 (GND), U8.8 (GND)
- net SWITCH_OUT: now reaches R_{SHUNT}1.1, U6.2 (IN-)
- net SWITCH_OUT: now also C_{BY}1.1, C_{IN_5}1.2, L1.1, U5.9 (VIN)
- net BATTERY: now reaches C_{CHARGE_OUT}1.1, U1.5 (BAT)
- net BATTERY: now also J3.2 (Pin_2), R_{SHUNT}1.2, SW1.2 (B), U5.2 (EN), U6.1 (IN+)
- removed net BATTERY+: C_{BY}1.1, C_{IN_5}1.2, L1.1, R_{SHUNT}1.2, U5.2 (EN), U5.9 (VIN), U6.1 (IN+)

Commit message: Added the zip into additional componenets of the missing footprint, Maybe you'll have better luck
Parts:
- D3, D4: footprint (none) -> Diode_SMD:D_SMA
- L2, L4: footprint (none) -> Inductor_SMD:L_0603_1608Metric
- Q3, Q4: footprint Package_TO_SOT_SMD:SOT-23 -> Package_TO_SOT_SMD:SOT-23-3
- U6: footprint INA219AIDCNR:SOT65P280X145-8N -> Package_TO_SOT_SMD:SOT-23-8
Changed lines of the file:
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@@
 			)
 		)
-		(property "Footprint" ""
+		(property "Footprint" "Diode_SMD:D_SMA"
 			(at 182.88 301.244 0)
 			(effects
@@
 			)
 		)
-		(property "Footprint" ""
+		(property "Footprint" "Inductor_SMD:L_0603_1608Metric"
 			(at 154.686 345.44 0)
 			(effects
@@
 			)
 		)
-		(property "Footprint" "Package_TO_SOT_SMD:SOT-23"
+		(property "Footprint" "Package_TO_SOT_SMD:SOT-23-3"
 			(at 76.2 49.53 0)
 			(effects
@@
 			)
 		)
-		(property "Footprint" "Package_TO_SOT_SMD:SOT-23"
+		(property "Footprint" "Package_TO_SOT_SMD:SOT-23-3"
 			(at 76.2 88.9 0)
 			(effects
@@
 			)
 		)
-		(property "Footprint" ""
+		(property "Footprint" "Inductor_SMD:L_0603_1608Metric"
 			(at 189.992 289.56 0)
 			(effects
@@
 			)
 		)
-		(property "Footprint" ""
+		(property "Footprint" "Diode_SMD:D_SMA"
 			(at 147.574 357.124 0)
 			(effects
@@
 			)
 		)
-		(property "Footprint" "INA219AIDCNR:SOT65P280X145-8N"
+		(property "Footprint" "Package_TO_SOT_SMD:SOT-23-8"
 			(at 373.38 146.05 0)
 			(effects

Commit message: save
Parts:
- J1: now left out of the parts list
- J3: now not fitted; now left out of the parts list
- L1: value L -> 1.2uH
Other:
- note added: "JST Connecter"
Changed lines of the file:
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@@
 	)
 	(rectangle
+		(start 299.72 263.525)
+		(end 369.57 289.56)
+		(stroke
+			(width 0)
+			(type dash)
+			(color 0 0 0 1)
+		)
+		(fill
+			(type none)
+		)
+	)
+	(rectangle
 		(start 13.335 329.184)
 		(end 231.775 378.46)
@@
 		)
 	)
+	(text "JST Connecter"
+		(exclude_from_sim no)
+		(at 345.948 286.512 0)
+		(effects
+			(font
+				(size 1.5 1.5)
+				(color 0 0 0 1)
+			)
+			(justify left bottom)
+		)
+	)
 	(text "Must handle 16V (min)\nX7R ceramic capacitor"
 		(exclude_from_sim no)
@@
 	(wire
 		(pts
-			(xy 383.54 210.82) (xy 391.16 210.82)
+			(xy 321.31 278.13) (xy 328.93 278.13)
 		)
 		(stroke
@@
 	(wire
 		(pts
-			(xy 387.35 208.28) (xy 391.16 208.28)
+			(xy 325.12 275.59) (xy 328.93 275.59)
 		)
 		(stroke
@@
 	)
 	(label "BATTERY"
-		(at 383.54 210.82 0)
+		(at 321.31 278.13 0)
 		(effects
 			(font
@@
 			)
 		)
-		(property "Value" "L"
+		(property "Value" "1.2uH"
 			(at 110.49 250.19 90)
 			(effects
@@
 		(lib_name "GND_2")
 		(lib_id "power:GND")
-		(at 387.35 208.28 180)
+		(at 325.12 275.59 180)
 		(unit 1)
 		(exclude_from_sim no)
@@
 		(fields_autoplaced yes)
 		(property "Reference" "#PWR030"
-			(at 387.35 201.93 0)
+			(at 325.12 269.24 0)
 			(effects
 				(font
@@
 		)
 		(property "Value" "GND"
-			(at 387.35 203.2 0)
+			(at 325.12 270.51 0)
 			(effects
 				(font
@@
 		)
 		(property "Footprint" ""
-			(at 387.35 208.28 0)
+			(at 325.12 275.59 0)
 			(effects
 				(font
@@
 		)
 		(property "Datasheet" ""
-			(at 387.35 208.28 0)
+			(at 325.12 275.59 0)
 			(effects
 				(font
@@
 		)
 		(property "Description" "Power symbol creates a global label with name \"GND\" , ground"
-			(at 387.35 208.28 0)
+			(at 325.12 275.59 0)
 			(effects
 				(font
@@
 	(symbol
 		(lib_id "Connector_Generic:Conn_01x02")
-		(at 396.24 208.28 0)
+		(at 334.01 275.59 0)
 		(unit 1)
 		(exclude_from_sim no)
-		(in_bom yes)
+		(in_bom no)
 		(on_board yes)
-		(dnp no)
+		(dnp yes)
 		(fields_autoplaced yes)
 		(property "Reference" "J3"
-			(at 399.415 208.28 0)
+			(at 337.185 275.59 0)
 			(effects
 				(font
@@
 		)
 		(property "Value" "Conn_01x02"
-			(at 399.415 210.82 0)
+			(at 337.185 278.13 0)
 			(effects
 				(font
@@
 		)
 		(property "Footprint" "Connector_JST:JST_PH_S2B-PH-K_1x02_P2.00mm_Horizontal"
-			(at 396.24 208.28 0)
+			(at 334.01 275.59 0)
 			(effects
 				(font
@@
 		)
 		(property "Datasheet" "~"
-			(at 396.24 208.28 0)
+			(at 334.01 275.59 0)
 			(effects
 				(font
@@
 		)
 		(property "Description" ""
-			(at 396.24 208.28 0)
+			(at 334.01 275.59 0)
 			(effects
 				(font
@@
 		(unit 1)
 		(exclude_from_sim no)
-		(in_bom yes)
+		(in_bom no)
 		(on_board yes)
 		(dnp yes)
