File: Micro-Mouse Power Subsystem.kicad_sch (KiCad schematic)
At the start: 81 parts, among them J1 Pin Header, J2 TYPE-C-31-M-12, J3 Conn_01x02, Q1 2N7002, Q2 AO3401A, Q3 AO3400A, Q4 AO3400A, Q5 AO3401A, SW1 SW_SPDT, U1 TP4056-42-ESOP8, U2 brushed DC motors, U3 auxiliary motors, U4 HUSB237-AA001-DN06R, U5 TPS61088RHLR, U6 INA219AIDCNR, U7 XL1509-3.3, U8 XL1509-5.0

Commit message: Added all my test points (as well as missing input for my charging circuit -- wild that i missed it
Parts:
- added TP10: SDA, symbol Connector:TestPoint
- added TP11: BATTERY_REG, symbol Connector:TestPoint
- added TP12: SWITCH_OUT_REG, symbol Connector:TestPoint
- added TP13: 5V_REG, symbol Connector:TestPoint
- added TP14: FB_5V, symbol Connector:TestPoint
- added TP15: 3V3_REG, symbol Connector:TestPoint
- added TP16: 5V_REG2, symbol Connector:TestPoint
- added TP17: 9V_CHRG, symbol Connector:TestPoint
- added TP18: 5V_CHRG, symbol Connector:TestPoint
- added TP19: FB_9V, symbol Connector:TestPoint
- added TP20: 5V_BAT_CHRG, symbol Connector:TestPoint
- added TP21: BATTERY_CHRG, symbol Connector:TestPoint
- added TP22: PROG, symbol Connector:TestPoint
- added TP23: CHRG_STDBY, symbol Connector:TestPoint
- added TP24: FAST_CHARGE, symbol Connector:TestPoint
- added TP6: BATTERY_MON, symbol Connector:TestPoint
- added TP7: SWITCH_OUT_MON, symbol Connector:TestPoint
- added TP8: 3V3_MON, symbol Connector:TestPoint
- added TP9: SCL, symbol Connector:TestPoint
Connections:
- net 3.3V_OUT: now also TP15.1, TP8.1
- net 5V_BAT_CHARGE: now also C_{CHARGE_IN}1.1, U1.4 (V_{CC}), U1.8 (CE), TP18.1, TP19.1, TP20.1
- net 5V_OUT: now also TP13.1, TP16.1
- net 9V_INPUT: now also TP17.1
- net BATTERY: now also TP11.1, TP21.1, TP6.1
- net FAST_CHARGE_CTRL: now also TP24.1
- net FB: now also TP14.1
- net GND: now also TP23.1
- net SWITCH_OUT: now also TP12.1, TP7.1
- net at R_{PROG}1.1, R_{PROG}2.1, U1.2 (PROG): now also TP22.1
- net at R_{SCL}1.1, U6.5 (SCL): now also TP9.1
- net at R_{SDA}1.2, U6.6 (SDA): now also TP10.1
Other:
- moved on the sheet: C_{CHARGE_OUT}1

Commit message: pcb sections
Parts:
- C10, C_{IN_3.3}1, C_{IN_3.3}2, C_{IN_3.3}3, C_{OUT_3.3}1, C_{OUT_3.3}2, C_{OUT_3.3}3, D3, L2, U7: Group (none) -> VOLT_REG_pt2
- C3, C4, C5, R5, R6, TP3, U2: Group (none) -> MOTOR_1
- C6, C7, C8, R7, R8, TP4, U3: Group (none) -> MOTOR_2
- C9, J2, R9, TP5, U4: Group (none) -> USBC
- C_{1}1, C_{IN}1, C_{IN}2, C_{IN}3, C_{OUT}1, C_{OUT}2, C_{OUT}3, D4, L4, U8: Group (none) -> STP_DWN
- C_{BOOT}1, C_{BY}1, C_{COMP}1, C_{IN_5}1, C_{OUT}4, C_{OUT}5, C_{OUT}6, C_{SS}1, L1, R_{COMP}1, R_{FB}1, R_{FB}2, R_{FSW}1, R_{FSW}2, R_{ILIM}1, U5: Group (none) -> VOLT_REG
- C_{BYPASS}1, R_{SCL}1, R_{SDA}1, R_{SHUNT}1, U6: Group (none) -> BATTERY_MONITORING
- C_{CHARGE_IN}1, C_{CHARGE_OUT}1, Q1, R_{LIMIT}1, R_{PROG}1, R_{PROG}2, R_{PULL_DOWN}1, U1: Group (none) -> BATTERY_CHARGING
- J1: Group (none) -> PIN_H
- J3: Group (none) -> BATT_CONN
- Q2, Q3, R1, R2, TP1: Group (none) -> EXT_LOAD_SWITCH_1
- Q4, Q5, R3, R4, TP2: Group (none) -> EXT_LOAD_SWITCH_2
- SW1: Group (none) -> SWITCH
- TP10, TP6, TP7, TP8, TP9: footprint (none) -> TestPoint:TestPoint_Pad_1.5x1.5mm; Group (none) -> BATTERY_MONITORING
- TP11, TP12, TP13, TP14: footprint (none) -> TestPoint:TestPoint_Pad_1.5x1.5mm; Group (none) -> VOLT_REG
- TP15, TP16: footprint (none) -> TestPoint:TestPoint_Pad_1.5x1.5mm; Group (none) -> VOLT_REG_pt2
- TP17, TP18, TP19: footprint (none) -> TestPoint:TestPoint_Pad_1.5x1.5mm; Group (none) -> STP_DWN
- TP20, TP21, TP22, TP23, TP24: footprint (none) -> TestPoint:TestPoint_Pad_1.5x1.5mm; Group (none) -> BATTERY_CHARGING

Commit message: updated pcb layout
Parts:
- C2: renamed from C_{IN}1; footprint Capacitor_SMD:C_1210_3225Metric -> Capacitor_SMD:C_1206_3216Metric
- C3: renamed from C_{IN}2; footprint Capacitor_SMD:C_1210_3225Metric -> Capacitor_SMD:C_1206_3216Metric
- TP10: renamed from TP16; value 5V_REG2 -> 5V_OUT
- TP16: renamed from TP13; value 5V_REG -> 5V_VOUT
- renumbered C_{CHARGE_IN}1 to C1, C_{IN_3.3}2 to C10, C_{IN_3.3}3 to C11, C10 to C12, C_{OUT}1 to C13, C_{OUT}2 to C14, C_{BOOT}1 to C15, C_{SS}1 to C16, C_{OUT}3 to C17, C_{OUT}4 to C18, C_{OUT_3.3}1 to C19, C_{OUT}5 to C20, C5 to C21, C6 to C22, C_{COMP}1 to C23, C_{OUT_3.3}2 to C24, C_{OUT}6 to C25, C_{OUT_3.3}3 to C26, C3 to C27, C7 to C28, C8 to C29, C4 to C30, C9 to C31, C_{BYPASS}1 to C32, C_{BY}1 to C4, C_{IN}3 to C5, C_{CHARGE_OUT}1 to C6, C_{IN_5}1 to C7, C_{IN_3.3}1 to C8, C_{1}1 to C9, D4 to D1, D3 to D2, J3 to J2, J2 to J3, L4 to L2, L2 to L3, Q3 to Q1, Q4 to Q2, Q2 to Q3, Q5 to Q4, Q1 to Q5, R2 to R1, R_{FSW}2 to R10, R_{ILIM}1 to R11, R5 to R12, R6 to R13, R7 to R14, R8 to R15, R_{COMP}1 to R16, R_{FB}1 to R17, R_{FB}2 to R18, R_{SHUNT}1 to R19, R3 to R2, R_{SCL}1 to R20, R_{SDA}1 to R21, R9 to R22, R1 to R3, R_{LIMIT}1 to R5, R_{PROG}1 to R6, R_{PULL_DOWN}1 to R7, R_{PROG}2 to R8, R_{FSW}1 to R9, TP20 to TP1, TP14 to TP12, TP19 to TP13, TP18 to TP14, TP3 to TP17, TP4 to TP18, TP6 to TP19, TP23 to TP2, TP7 to TP20, TP9 to TP21, TP10 to TP22, TP5 to TP23, TP8 to TP24, TP24 to TP3, TP2 to TP4, TP1 to TP5, TP17 to TP6, TP22 to TP7, TP21 to TP8, TP12 to TP9, U8 to U2, U5 to U3, U7 to U4, U2 to U5, U3 to U6, U6 to U7, U4 to U8
Connections:
- net Battery  is gone; now on net BATTERY: J1.14 (Pin_14)
- net Motor2_A_OUT is gone; now on net MOTOR2_A_OUT: J1.2 (Pin_2)
- net Motor2_B_OUT is gone; now on net MOTOR2_B_OUT: J1.1 (Pin_1)
- net Motor4_A_OUT is gone; now on net MOTOR4_A_OUT: J1.3 (Pin_3)
- net Motor4_B_OUT is gone; now on net MOTOR4_B_OUT: J1.5 (Pin_5)
- net 5V Out : no longer J1.20 (Pin_20), Q3.3 (D), Q4.3 (D), R3.1, R4.1
- net 5V_OUT: now also J1.20 (Pin_20), Q3.3 (D), Q4.3 (D), R3.1, R4.1
- no-connect marks 0 -> 3
